File: Upgrade_Parts/BLV_Toolhead_PCB/accelerometer.kicad_sch (KiCad schematic)
At the start: 13 parts, among them J10 RB1-125B8G1A, U1 SN65LVDS2, U2 SN65LVDS1, U3 SN65LVDS1, U4 LIS3DH

Commit message: replaced lvds drver
Parts:
- removed C4: 100n, symbol Device:C
- removed U1: SN65LVDS2, Package_TO_SOT_SMD:SOT-23-5, symbol toolhead:SN65LVDS2
- removed U2, U3: SN65LVDS1, Package_TO_SOT_SMD:SOT-23-5, symbol toolhead:SN65LVDS1
- added R4: 100, Resistor_SMD:R_0402_1005Metric, symbol Device:R
- added U1: DS90LV028AQ, Package_SO:SOIC-8_3.9x4.9mm_P1.27mm, symbol toolhead:DS90LV028AQ
- added U2: DS90LV027A, Package_SO:SOIC-8_3.9x4.9mm_P1.27mm, symbol Interface:DS90LV027A
- C2, C3: footprint (none) -> Capacitor_SMD:C_0402_1005Metric
- C4: renamed from C5; footprint (none) -> Capacitor_SMD:C_0402_1005Metric
- C5: renamed from C6; footprint (none) -> Capacitor_SMD:C_0603_1608Metric
- R1, R2, R3: footprint (none) -> Resistor_SMD:R_0402_1005Metric
- renumbered U4 to U3
Connections:
- net +3V3: now also U1.8 (VCC), U2.1 (VCC)
- net GND: now also U1.5 (GND), U2.4 (GND)
- net INT1: now also U2.3 (DI2)
- net INT1_N: now also U2.5 (DO-2)
- net INT1_P: now also U2.6 (DO+2)
- net SPI_MISO: now also U1.7 (RO1)
- net SPI_MISO_N: now also U2.8 (DO-1)
- net SPI_MISO_P: now also U2.7 (DO+1)
- net SPI_MOSI: now also U2.2 (DI1)
- net SPI_MOSI_N: now also U1.1 (RI1-)
- net SPI_MOSI_P: now also U1.2 (RI1+)
- new net: R4.1, U1.3 (RI2+)
- new net: R4.2, U1.4 (RI2-)
- no-connect marks 8 -> 9
Other:
- note removed: "5V!!!"
- moved on the sheet: C2, C3, J10, R1, R2, R3
